File: test/cli/big/reference/pcbs/_export.kicad_pcb (KiCad board)
At the start: 2 copper layers, 0 parts

Commit message: Apply soundmonster's footprint changes
Add a separate netclass with wider traces for power

Add option to skip key-based footprints in PCBs

First try at flipping the silkscreen for promicro

Mirror text

Tighten TRRS stab poles

Also fix the reverse TRRS footprint as it doesn't make sense the way it is

Fix TRRS docs

Allow using more than one TRRS on a board

Add a simple text footprint

Finalize text footprint

Add battery pins to promicro

Add battery nets to power netclass

Fix net naming for battery pins

Allow using the simple two-pin through hole button
Other:
- net class Power added: clearance 0.2, trace_width 0.5, via_dia 0.8, via_drill 0.4
Changed lines of the file:
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@@
     (add_net "")
   )
+  (net_class Power "This is the power net class."
+    (clearance 0.2)
+    (trace_width 0.5)
+    (via_dia 0.8)
+    (via_drill 0.4)
+    (uvia_dia 0.3)
+    (uvia_drill 0.1)
+  )
 )
